File: i2cio/AVR.sch (KiCad schematic (older format))
At the start: 22 parts, among them CON2 AVR-ISP-6, CON3 AVR-JTAG-10, IC1 ATMEGA32-A, P10 CONN_01X03, P11 CONN_01X03, P4 CONN_01X11, P5 CONN_01X11, P6 CONN_01X11, P7 CONN_01X11, SW1 Tactile_switch, Y1 16MHz

Commit message: pcb almost done
Parts:
- added D2: LED, amol_parts_footprints:0805_HandSoldering, symbol LED
- added R2: 1K, amol_parts_footprints:0805_HandSoldering, symbol R
- C10, C11, C12, C5, C6, C7, C8, C9, D1, R1: footprint (none) -> amol_parts_footprints:0805_HandSoldering
- CON2: footprint AVR-ISP-6 -> Pin_Headers:Pin_Header_Straight_2x03
- CON3: footprint AVR-JTAG-10 -> Pin_Headers:Pin_Header_Straight_2x05
- IC1: footprint TQFP44 -> amol_parts_footprints:TQFP-44-1EP_10x10mm_Pitch0.8mm
- L1: footprint (none) -> amol_parts_footprints:1206_HandSoldering
- P10, P11: footprint (none) -> Pin_Headers:Pin_Header_Angled_1x03
- P4, P5, P6, P7: footprint (none) -> Pin_Headers:Pin_Header_Straight_1x11
- SW1: footprint (none) -> amol_parts_footprints:SW_PUSH_SMALL
- Y1: footprint (none) -> Crystals:Crystal_HC49-U_Vertical
Connections:
- net labels removed: Reset
- wire segments 213 -> 224
