File: i2cio/analog.sch (KiCad schematic (older format))
At the start: 10 parts, among them P8 CONN_01X08, P9 CONN_01X08, U3 MCP4361, U4 MCP4361, U5 OPA4350, U6 OPA4350

Commit message: pcb almost done
Parts:
- removed P8, P9: CONN_01X08, symbol CONN_01X08
- added P8: CONN_02X08, Pin_Headers:Pin_Header_Straight_2x08, symbol CONN_02X08
- C13, C14, C15, C16: footprint (none) -> amol_parts_footprints:0805_HandSoldering
- U3, U4: footprint (none) -> amol_parts_footprints:TSSOP-20_4.4x6.5mm_Pitch0.65mm
- U5, U6: footprint (none) -> amol_parts_footprints:SOIC-14_3.9x8.7mm_Pitch1.27mm
Connections:
- wire segments 173 -> 177
Changed lines of the file:
@@
 $Descr A4 11693 8268
 encoding utf-8
-Sheet 4 4
+Sheet 4 5
 Title ""
 Date ""
@@
 F 0 "U5" H 3600 2100 60  0000 C CNN
 F 1 "OPA4350" H 3600 2900 60  0000 C CNN
-F 2 "" H 3600 2350 60  0000 C CNN
+F 2 "amol_parts_footprints:SOIC-14_3.9x8.7mm_Pitch1.27mm" H 3600 2350 60  0001 C CNN
 F 3 "" H 3600 2350 60  0000 C CNN
 	1    3600 2500
@@
 F 0 "U3" H 1750 1950 60  0000 C CNN
 F 1 "MCP4361" H 1750 3050 60  0000 C CNN
-F 2 "" H 1750 2500 60  0000 C CNN
+F 2 "amol_parts_footprints:TSSOP-20_4.4x6.5mm_Pitch0.65mm" H 1750 2500 60  0001 C CNN
 F 3 "" H 1750 2500 60  0000 C CNN
 	1    1750 2500
@@
 Connection ~ 700  2750
 $Comp
-L GNDA #PWR050
+L GNDA #PWR048
 U 1 1 56063093
 P 2650 3500
-F 0 "#PWR050" H 2650 3250 50  0001 C CNN
+F 0 "#PWR048" H 2650 3250 50  0001 C CNN
 F 1 "GNDA" H 2650 3350 50  0000 C CNN
 F 2 "" H 2650 3500 60  0000 C CNN
@@
 F 0 "U6" H 3650 5650 60  0000 C CNN
 F 1 "OPA4350" H 3650 6450 60  0000 C CNN
-F 2 "" H 3650 5900 60  0000 C CNN
+F 2 "amol_parts_footprints:SOIC-14_3.9x8.7mm_Pitch1.27mm" H 3650 5900 60  0001 C CNN
 F 3 "" H 3650 5900 60  0000 C CNN
 	1    3650 6050
@@
 F 0 "U4" H 1800 5500 60  0000 C CNN
 F 1 "MCP4361" H 1800 6600 60  0000 C CNN
-F 2 "" H 1800 6050 60  0000 C CNN
+F 2 "amol_parts_footprints:TSSOP-20_4.4x6.5mm_Pitch0.65mm" H 1800 6050 60  0001 C CNN
 F 3 "" H 1800 6050 60  0000 C CNN
 	1    1800 6050
@@
 Connection ~ 750  6300
 $Comp
-L GNDA #PWR051
+L GNDA #PWR049
 U 1 1 56064318
 P 2700 7050
-F 0 "#PWR051" H 2700 6800 50  0001 C CNN
+F 0 "#PWR049" H 2700 6800 50  0001 C CNN
 F 1 "GNDA" H 2700 6900 50  0000 C CNN
 F 2 "" H 2700 7050 60  0000 C CNN
@@
 	600  2650 600  2550
 $Comp
-L +3V3 #PWR052
+L +3V3 #PWR050
 U 1 1 56064D8B
 P 600 2550
-F 0 "#PWR052" H 600 2400 50  0001 C CNN
+F 0 "#PWR050" H 600 2400 50  0001 C CNN
 F 1 "+3V3" H 600 2690 50  0000 C CNN
 F 2 "" H 600 2550 60  0000 C CNN
@@
 $EndComp
 $Comp
-L +3V3 #PWR053
+L +3V3 #PWR051
 U 1 1 56064DA9
 P 600 6100
-F 0 "#PWR053" H 600 5950 50  0001 C CNN
+F 0 "#PWR051" H 600 5950 50  0001 C CNN
 F 1 "+3V3" H 600 6240 50  0000 C CNN
 F 2 "" H 600 6100 60  0000 C CNN
@@
 	5000 6050 5000 6950
 $Comp
-L +5V #PWR054
+L +5V #PWR052
 U 1 1 5606524E
 P 2850 6150
-F 0 "#PWR054" H 2850 6000 50  0001 C CNN
+F 0 "#PWR052" H 2850 6000 50  0001 C CNN
 F 1 "+5V" H 2850 6290 50  0000 C CNN
 F 2 "" H 2850 6150 60  0000 C CNN
@@
 $EndComp
 $Comp
-L +5V #PWR055
+L +5V #PWR053
 U 1 1 5606526C
 P 2800 2600
-F 0 "#PWR055" H 2800 2450 50  0001 C CNN
+F 0 "#PWR053" H 2800 2450 50  0001 C CNN
 F 1 "+5V" H 2800 2740 50  0000 C CNN
 F 2 "" H 2800 2600 60  0000 C CNN
@@
 	2900 6050 3100 6050
 Wire Wire Line
-	7050 2800 7900 2800
-Wire Wire Line
-	7900 2900 7050 2900
-Wire Wire Line
-	7900 3000 7050 3000
-Wire Wire Line
-	7900 3100 7050 3100
-Wire Wire Line
-	7050 3200 7900 3200
-Wire Wire Line
-	7900 3300 7050 3300
-Wire Wire Line
-	7900 3400 7050 3400
-Wire Wire Line
-	7900 3500 7050 3500
+	7050 2800 7950 2800
+Wire Wire Line
+	7950 2900 7050 2900
+Wire Wire Line
+	7950 3000 7050 3000
+Wire Wire Line
+	7950 3100 7050 3100
+Wire Wire Line
+	7050 3200 7950 3200
+Wire Wire Line
+	7950 3300 7050 3300
+Wire Wire Line
+	7950 3400 7050 3400
+Wire Wire Line
+	7950 3500 7050 3500
 Text Label 7100 2800 0    60   ~ 0
 Amp1_IN_A
@@
 Amp2_IN_D
 Wire Wire Line
-	8900 3500 9250 3500
-Wire Wire Line
-	8900 3500 8900 3700
-$Comp
-L GNDA #PWR056
+	8450 3500 8800 3500
+Wire Wire Line
+	8800 3500 8800 3700
+$Comp
+L GNDA #PWR054
 U 1 1 5606657C
-P 8900 3700
-F 0 "#PWR056" H 8900 3450 50  0001 C CNN
-F 1 "GNDA" H 8900 3550 50  0000 C CNN
-F 2 "" H 8900 3700 60  0000 C CNN
-F 3 "" H 8900 3700 60  0000 C CNN
-	1    8900 3700
-	1    0    0    -1
+P 8800 3700
+F 0 "#PWR054" H 8800 3450 50  0001 C CNN
+F 1 "GNDA" H 8800 3550 50  0000 C CNN
+F 2 "" H 8800 3700 60  0000 C CNN
+F 3 "" H 8800 3700 60  0000 C CNN
+	1    8800 3700
+	-1   0    0    -1
 $EndComp
 Text GLabel 4100 650  2    60   Input ~ 0
@@
 F 0 "C15" H 8100 1250 50  0000 L CNN
 F 1 "100nF" H 8000 1050 50  0000 L CNN
-F 2 "" H 8288 1000 30  0000 C CNN
+F 2 "amol_parts_footprints:0805_HandSoldering" H 8288 1000 30  0001 C CNN
 F 3 "" H 8250 1150 60  0000 C CNN
 	1    8250 1150
@@
 F 0 "C16" H 8450 1250 50  0000 L CNN
 F 1 "100nF" H 8475 1050 50  0000 L CNN
-F 2 "" H 8488 1000 30  0000 C CNN
+F 2 "amol_parts_footprints:0805_HandSoldering" H 8488 1000 30  0001 C CNN
 F 3 "" H 8450 1150 60  0000 C CNN
 	1    8450 1150
@@
 F 0 "C14" H 7000 1250 50  0000 L CNN
 F 1 "100nF" H 6900 1050 50  0000 L CNN
-F 2 "" H 7188 1000 30  0000 C CNN
+F 2 "amol_parts_footprints:0805_HandSoldering" H 7188 1000 30  0001 C CNN
 F 3 "" H 7150 1150 60  0000 C CNN
 	1    7150 1150
@@
 F 0 "C13" H 7350 1250 50  0000 L CNN
 F 1 "100nF" H 7400 1050 50  0000 L CNN
-F 2 "" H 7388 1000 30  0000 C CNN
+F 2 "amol_parts_footprints:0805_HandSoldering" H 7388 1000 30  0001 C CNN
 F 3 "" H 7350 1150 60  0000 C CNN
 	1    7350 1150
@@
 	8250 1000 8450 1000
 $Comp
-L GNDA #PWR057
+L GNDA #PWR055
 U 1 1 5606823B
-P 8350 1300
-F 0 "#PWR057" H 8350 1050 50  0001 C CNN
-F 1 "GNDA" H 8350 1150 50  0000 C CNN
-F 2 "" H 8350 1300 60  0000 C CNN
-F 3 "" H 8350 1300 60  0000 C CNN
-	1    8350 1300
-	1    0    0    -1
-$EndComp
-$Comp
-L GNDA #PWR058
+P 8350 1450
+F 0 "#PWR055" H 8350 1200 50  0001 C CNN
+F 1 "GNDA" H 8350 1300 50  0000 C CNN
+F 2 "" H 8350 1450 60  0000 C CNN
+F 3 "" H 8350 1450 60  0000 C CNN
+	1    8350 1450
+	1    0    0    -1
+$EndComp
+$Comp
+L GNDA #PWR056
 U 1 1 56068268
-P 7250 1300
-F 0 "#PWR058" H 7250 1050 50  0001 C CNN
-F 1 "GNDA" H 7250 1150 50  0000 C CNN
-F 2 "" H 7250 1300 60  0000 C CNN
-F 3 "" H 7250 1300 60  0000 C CNN
-	1    7250 1300
-	1    0    0    -1
-$EndComp
-$Comp
-L +5V #PWR059
+P 7250 1450
+F 0 "#PWR056" H 7250 1200 50  0001 C CNN
+F 1 "GNDA" H 7250 1300 50  0000 C CNN
+F 2 "" H 7250 1450 60  0000 C CNN
+F 3 "" H 7250 1450 60  0000 C CNN
+	1    7250 1450
+	1    0    0    -1
+$EndComp
+$Comp
+L +5V #PWR057
 U 1 1 56068287
-P 7250 1000
-F 0 "#PWR059" H 7250 850 50  0001 C CNN
-F 1 "+5V" H 7250 1140 50  0000 C CNN
-F 2 "" H 7250 1000 60  0000 C CNN
-F 3 "" H 7250 1000 60  0000 C CNN
-	1    7250 1000
-	1    0    0    -1
-$EndComp
-$Comp
-L +3V3 #PWR060
+P 7250 850
+F 0 "#PWR057" H 7250 700 50  0001 C CNN
+F 1 "+5V" H 7250 990 50  0000 C CNN
+F 2 "" H 7250 850 60  0000 C CNN
+F 3 "" H 7250 850 60  0000 C CNN
+	1    7250 850
+	1    0    0    -1
+$EndComp
+$Comp
+L +3V3 #PWR058
 U 1 1 560682AD
-P 8350 1000
-F 0 "#PWR060" H 8350 850 50  0001 C CNN
-F 1 "+3V3" H 8350 1140 50  0000 C CNN
-F 2 "" H 8350 1000 60  0000 C CNN
-F 3 "" H 8350 1000 60  0000 C CNN
-	1    8350 1000
-	1    0    0    -1
-$EndComp
-$Comp
-L CONN_01X08 P8
-U 1 1 5606B2F7
-P 8100 3150
-F 0 "P8" H 8100 3600 50  0000 C CNN
-F 1 "CONN_01X08" V 8200 3150 50  0000 C CNN
-F 2 "" H 8100 3150 60  0000 C CNN
-F 3 "" H 8100 3150 60  0000 C CNN
-	1    8100 3150
-	1    0    0    -1
-$EndComp
-$Comp
-L CONN_01X08 P9
-U 1 1 5606B451
-P 9450 3150
-F 0 "P9" H 9450 3600 50  0000 C CNN
-F 1 "CONN_01X08" V 9550 3150 50  0000 C CNN
-F 2 "" H 9450 3150 60  0000 C CNN
-F 3 "" H 9450 3150 60  0000 C CNN
-	1    9450 3150
-	1    0    0    -1
-$EndComp
-Wire Wire Line
-	9050 2800 9050 3500
-Wire Wire Line
-	9050 2800 9250 2800
-Connection ~ 9050 3500
-Wire Wire Line
-	9250 3400 9050 3400
-Connection ~ 9050 3400
-Wire Wire Line
-	9050 3300 9250 3300
-Connection ~ 9050 3300
-Wire Wire Line
-	9250 3200 9050 3200
-Connection ~ 9050 3200
-Wire Wire Line
-	9050 3100 9250 3100
-Connection ~ 9050 3100
-Wire Wire Line
-	9250 3000 9050 3000
-Connection ~ 9050 3000
-Wire Wire Line
-	9050 2900 9250 2900
-Connection ~ 9050 2900
+P 8350 900
+F 0 "#PWR058" H 8350 750 50  0001 C CNN
+F 1 "+3V3" H 8350 1040 50  0000 C CNN
+F 2 "" H 8350 900 60  0000 C CNN
+F 3 "" H 8350 900 60  0000 C CNN
+	1    8350 900
+	1    0    0    -1
+$EndComp
+Wire Wire Line
+	8650 2800 8650 3500
+Wire Wire Line
+	8650 2800 8450 2800
+Connection ~ 8650 3500
+Wire Wire Line
+	8450 3400 8650 3400
+Connection ~ 8650 3400
+Wire Wire Line
+	8650 3300 8450 3300
+Connection ~ 8650 3300
+Wire Wire Line
+	8450 3200 8650 3200
+Connection ~ 8650 3200
+Wire Wire Line
+	8650 3100 8450 3100
+Connection ~ 8650 3100
+Wire Wire Line
+	8450 3000 8650 3000
+Connection ~ 8650 3000
+Wire Wire Line
+	8650 2900 8450 2900
+Connection ~ 8650 2900
 Text GLabel 1000 2550 0    60   Input ~ 0
 MOSI
@@
 	1150 5900 1250 5900
 $Comp
-L PWR_FLAG #FLG061
+L PWR_FLAG #FLG059
 U 1 1 56074794
 P 2200 7050
-F 0 "#FLG061" H 2200 7145 50  0001 C CNN
+F 0 "#FLG059" H 2200 7145 50  0001 C CNN
 F 1 "PWR_FLAG" H 2200 7230 50  0000 C CNN
 F 2 "" H 2200 7050 60  0000 C CNN
@@
 	2200 7050 2200 6950
 Connection ~ 2200 6950
+$Comp
+L CONN_02X08 P8
+U 1 1 560758C5
+P 8200 3150
+F 0 "P8" H 8200 3600 50  0000 C CNN
+F 1 "CONN_02X08" V 8200 3150 50  0000 C CNN
+F 2 "Pin_Headers:Pin_Header_Straight_2x08" H 8200 1950 60  0001 C CNN
+F 3 "" H 8200 1950 60  0000 C CNN
+	1    8200 3150
+	1    0    0    -1
+$EndComp
+Wire Wire Line
+	7250 1000 7250 850
+Connection ~ 7250 1000
+Wire Wire Line
+	7250 1450 7250 1300
+Connection ~ 7250 1300
+Wire Wire Line
+	8350 1450 8350 1300
+Connection ~ 8350 1300
+Wire Wire Line
+	8350 1000 8350 900
+Connection ~ 8350 1000
 $EndSCHEMATC
