File: i2cio/i2cio.sch (KiCad schematic (older format))
At the start: 0 parts

Commit message: pcb almost done
Changed lines of the file:
@@
 $Descr A4 11693 8268
 encoding utf-8
-Sheet 1 4
+Sheet 1 5
 Title ""
 Date ""
@@
 F1 "analog.sch" 60
 $EndSheet
+$Sheet
+S 5000 3750 1500 1150
+U 5610330E
+F0 "groundpoints" 60
+F1 "groundpoints.sch" 60
+$EndSheet
 $EndSCHEMATC
