File: i2cio/power.sch (KiCad schematic (older format))
At the start: 10 parts, among them CON1 BARREL_JACK, P1 CONN_01X02, P2 CONN_01X03, P3 CONN_01X03, U1 LM2940, U2 LM3940

Commit message: pcb almost done
Parts:
- removed P2, P3: CONN_01X03, symbol CONN_01X03
- C1, C3: footprint (none) -> amol_parts_footprints:0805_HandSoldering
- C2, C4: footprint (none) -> amol_parts_footprints:Aluminum SMD Electrolytic Capacitor - Size C
- CON1: footprint (none) -> Connect:BARREL_JACK
- P1: footprint (none) -> Pin_Headers:Pin_Header_Straight_1x02
- U1, U2: footprint (none) -> TO_SOT_Packages_SMD:SOT-223
Changed lines of the file:
@@
 $Descr A4 11693 8268
 encoding utf-8
-Sheet 2 4
+Sheet 2 5
 Title ""
 Date ""
@@
 F 0 "P1" H 1450 1300 50  0000 C CNN
 F 1 "CONN_01X02" V 1550 1150 50  0000 C CNN
-F 2 "" H 1450 1150 60  0000 C CNN
+F 2 "Pin_Headers:Pin_Header_Straight_1x02" H 1450 1150 60  0001 C CNN
 F 3 "" H 1450 1150 60  0000 C CNN
 	1    1450 1150
@@
 F 0 "CON1" H 3200 1350 60  0000 C CNN
 F 1 "BARREL_JACK" H 3200 900 60  0000 C CNN
-F 2 "" H 3200 1100 60  0000 C CNN
+F 2 "Connect:BARREL_JACK" H 3200 1100 60  0001 C CNN
 F 3 "" H 3200 1100 60  0000 C CNN
 	1    3200 1100
@@
 F 0 "U2" H 4500 2904 60  0000 C CNN
 F 1 "LM3940" H 4350 3300 60  0000 C CNN
-F 2 "" H 4350 3100 60  0000 C CNN
+F 2 "TO_SOT_Packages_SMD:SOT-223" H 4350 3100 60  0001 C CNN
 F 3 "" H 4350 3100 60  0000 C CNN
 	1    4350 3100
@@
 F 0 "C3" H 3625 3300 50  0000 L CNN
 F 1 "0.47uF" H 3625 3100 50  0000 L CNN
-F 2 "" H 3638 3050 30  0000 C CNN
+F 2 "amol_parts_footprints:0805_HandSoldering" H 3638 3050 30  0001 C CNN
 F 3 "" H 3600 3200 60  0000 C CNN
 	1    3600 3200
@@
 F 0 "C4" H 4975 3300 50  0000 L CNN
 F 1 "100uF" H 4975 3100 50  0000 L CNN
-F 2 "" H 4950 3200 60  0000 C CNN
+F 2 "amol_parts_footprints:Aluminum SMD Electrolytic Capacitor - Size C" H 4950 3200 60  0001 C CNN
 F 3 "" H 4950 3200 60  0000 C CNN
 	1    4950 3200
@@
 F 0 "U1" H 1750 2904 60  0000 C CNN
 F 1 "LM2940" H 1600 3300 60  0000 C CNN
-F 2 "" H 1600 3100 60  0000 C CNN
+F 2 "TO_SOT_Packages_SMD:SOT-223" H 1600 3100 60  0001 C CNN
 F 3 "" H 1600 3100 60  0000 C CNN
 	1    1600 3100
@@
 F 0 "C1" H 1025 3350 50  0000 L CNN
 F 1 "0.47uF" H 1025 3150 50  0000 L CNN
-F 2 "" H 1038 3100 30  0000 C CNN
+F 2 "amol_parts_footprints:0805_HandSoldering" H 1038 3100 30  0001 C CNN
 F 3 "" H 1000 3250 60  0000 C CNN
 	1    1000 3250
@@
 F 0 "C2" H 2275 3350 50  0000 L CNN
 F 1 "100uF" H 2275 3150 50  0000 L CNN
-F 2 "" H 2250 3250 60  0000 C CNN
+F 2 "amol_parts_footprints:Aluminum SMD Electrolytic Capacitor - Size C" H 2250 3250 60  0001 C CNN
 F 3 "" H 2250 3250 60  0000 C CNN
 	1    2250 3250
@@
 External supply\n
 $Comp
-L CONN_01X03 P2
-U 1 1 5606A831
-P 1500 5650
-F 0 "P2" H 1500 5850 50  0000 C CNN
-F 1 "CONN_01X03" V 1600 5650 50  0000 C CNN
-F 2 "" H 1500 5650 60  0000 C CNN
-F 3 "" H 1500 5650 60  0000 C CNN
-	1    1500 5650
-	0    -1   -1   0
-$EndComp
-$Comp
-L CONN_01X03 P3
-U 1 1 5606AB36
-P 2250 5650
-F 0 "P3" H 2250 5850 50  0000 C CNN
-F 1 "CONN_01X03" V 2350 5650 50  0000 C CNN
-F 2 "" H 2250 5650 60  0000 C CNN
-F 3 "" H 2250 5650 60  0000 C CNN
-	1    2250 5650
-	0    -1   -1   0
-$EndComp
-$Comp
-L +3V3 #PWR011
-U 1 1 5606AD1A
-P 1350 6200
-F 0 "#PWR011" H 1350 6050 50  0001 C CNN
-F 1 "+3V3" H 1350 6340 50  0000 C CNN
-F 2 "" H 1350 6200 60  0000 C CNN
-F 3 "" H 1350 6200 60  0000 C CNN
-	1    1350 6200
-	1    0    0    -1
-$EndComp
-$Comp
-L +5V #PWR012
-U 1 1 5606AF40
-P 1600 6200
-F 0 "#PWR012" H 1600 6050 50  0001 C CNN
-F 1 "+5V" H 1600 6340 50  0000 C CNN
-F 2 "" H 1600 6200 60  0000 C CNN
-F 3 "" H 1600 6200 60  0000 C CNN
-	1    1600 6200
-	1    0    0    -1
-$EndComp
-$Comp
-L GND #PWR013
-U 1 1 5606AF68
-P 1100 6100
-F 0 "#PWR013" H 1100 5850 50  0001 C CNN
-F 1 "GND" H 1100 5950 50  0000 C CNN
-F 2 "" H 1100 6100 60  0000 C CNN
-F 3 "" H 1100 6100 60  0000 C CNN
-	1    1100 6100
-	1    0    0    -1
-$EndComp
-$Comp
-L +3V3 #PWR014
-U 1 1 5606B010
-P 2350 6200
-F 0 "#PWR014" H 2350 6050 50  0001 C CNN
-F 1 "+3V3" H 2350 6340 50  0000 C CNN
-F 2 "" H 2350 6200 60  0000 C CNN
-F 3 "" H 2350 6200 60  0000 C CNN
-	1    2350 6200
-	1    0    0    -1
-$EndComp
-$Comp
-L +5V #PWR015
-U 1 1 5606B016
-P 2600 6200
-F 0 "#PWR015" H 2600 6050 50  0001 C CNN
-F 1 "+5V" H 2600 6340 50  0000 C CNN
-F 2 "" H 2600 6200 60  0000 C CNN
-F 3 "" H 2600 6200 60  0000 C CNN
-	1    2600 6200
-	1    0    0    -1
-$EndComp
-$Comp
-L GND #PWR016
-U 1 1 5606B01C
-P 2100 6100
-F 0 "#PWR016" H 2100 5850 50  0001 C CNN
-F 1 "GND" H 2100 5950 50  0000 C CNN
-F 2 "" H 2100 6100 60  0000 C CNN
-F 3 "" H 2100 6100 60  0000 C CNN
-	1    2100 6100
-	1    0    0    -1
-$EndComp
-Wire Wire Line
-	1350 6200 1500 6200
-Wire Wire Line
-	1500 6200 1500 5850
-Wire Wire Line
-	1700 5900 1700 6250
-Wire Wire Line
-	1700 5900 1600 5900
-Wire Wire Line
-	1600 5900 1600 5850
-Wire Wire Line
-	1100 6100 1100 5900
-Wire Wire Line
-	1100 5900 1400 5900
-Wire Wire Line
-	1400 5900 1400 5850
-Wire Wire Line
-	2100 5900 2100 6100
-Wire Wire Line
-	2100 5900 2150 5900
-Wire Wire Line
-	2150 5900 2150 5850
-Wire Wire Line
-	2350 6200 2250 6200
-Wire Wire Line
-	2250 6200 2250 5850
-Wire Wire Line
-	2350 5850 2350 5950
-Wire Wire Line
-	2350 5950 2500 5950
-Wire Wire Line
-	2500 5950 2500 6250
-Wire Wire Line
-	2500 6250 2600 6250
-Wire Wire Line
-	2600 6250 2600 6200
-Wire Wire Line
-	1600 6200 1600 6250
-Wire Wire Line
-	1600 6250 1700 6250
-$Comp
-L PWR_FLAG #FLG017
+L PWR_FLAG #FLG011
 U 1 1 560708AF
 P 4150 1000
-F 0 "#FLG017" H 4150 1095 50  0001 C CNN
+F 0 "#FLG011" H 4150 1095 50  0001 C CNN
 F 1 "PWR_FLAG" H 4150 1180 50  0000 C CNN
 F 2 "" H 4150 1000 60  0000 C CNN
@@
 Wire Wire Line
 	3500 1200 3650 1200
+$Comp
+L GND #PWR012
+U 1 1 56108714
+P 1900 4650
+F 0 "#PWR012" H 1900 4400 50  0001 C CNN
+F 1 "GND" H 1900 4500 50  0000 C CNN
+F 2 "" H 1900 4650 60  0000 C CNN
+F 3 "" H 1900 4650 60  0000 C CNN
+	1    1900 4650
+	1    0    0    -1
+$EndComp
+$Comp
+L GNDA #PWR013
+U 1 1 56108738
+P 2200 4650
+F 0 "#PWR013" H 2200 4400 50  0001 C CNN
+F 1 "GNDA" H 2200 4500 50  0000 C CNN
+F 2 "" H 2200 4650 60  0000 C CNN
+F 3 "" H 2200 4650 60  0000 C CNN
+	1    2200 4650
+	1    0    0    -1
+$EndComp
+Wire Wire Line
+	1900 4650 1900 4600
+Wire Wire Line
+	1900 4600 2200 4600
+Wire Wire Line
+	2200 4600 2200 4650
 $EndSCHEMATC
